File: layout/onecolor stripe/v1.0/universal.sch (EAGLE design)
At the start: 39 parts, among them IC2 FT232RL, Q1 PSMN2R0-30YL, Q2 PSMN2R0-30YL, Q3 PSMN2R0-30YL, Q4 PSMN2R0-30YL, T1 BC848, T2 BC848, X1 6PIN_MDF6-6DP-3.5DS, X4 1PIN_SCHRAUBKLEMME, X5 1PIN_SCHRAUBKLEMME, X6 1PIN_SCHRAUBKLEMME

Commit message: Finished layout for 4*RGBW stripe v1.0
Parts:
- removed U$2: ESP8266, ESP8266:ESP8266
- removed U$40: USB-B, sid:USB-B
- removed U2: (no value), adafruit:PCA9685
- added C10: 100n, rcl:C-EUC0603
- added C11, C12, C13: 100u, cap-master:CP-7343-TE-D
- added D1: MBRS240, diode:MBRS130LT3
- added Q10, Q11, Q12, Q13, Q14, Q15, Q16, Q5, Q6, Q7, Q8, Q9: PSMN2R0-30YL, transistor-yaala:PSMN2R0-30YL
- added R10, R11, R12, R13, R14, R15, R16, R17, R18, R24, R25, R9: 1k, rcl-2:R-EU_R0603
- added ST1, ST2, ST3: 5PIN_STIFTLEISTE_1,27MM, con-yaala:5PIN_STIFTLEISTE_1,27MM
- added U$1: ESP8266, ESP8266:ESP8266
- added U1: (no value), adafruit:PCA9685
- added X10, X11, X12, X13, X15, X16, X17, X18, X20, X21, X22, X23: 1PIN_SCHRAUBKLEMME, con-yaala:1PIN_SCHRAUBKLEMME
- added X14, X19, X2, X9: 6PIN_MDF6-6DP-3.5DS, con-yaala:6PIN_MDF6-6DP-3.5DS
- added X7, X8: 10PIN_LEOTRONICS_1296-10, con-yaala:10PIN_LEOTRONICS_1296-10
- C3: value 22p -> 100n
- C4: value 22p -> 100u; device rcl:C-EUC0603 -> cap-master:CP-7343-TE-D
- C6: value 100u -> 100n; device cap-master:CP-7343-TE-D -> rcl:C-EUC0603
- C7, C8: value 100n -> 22p
- R1, R2, R5, R6, R7: value 1k -> 10k
- R19, R20, R21, R22, R23: value 10k -> 1k
- X1: value 6PIN_MDF6-6DP-3.5DS -> USB-B; device con-yaala:6PIN_MDF6-6DP-3.5DS -> sid:USB-B
Connections:
- removed net B: Q3.G, R7.1
- removed net G: Q2.G, R6.1
- removed net R: Q1.G, R5.1
- removed net W: Q4.G, R8.1
- new net B1: R13.1, U1.PWM2, X7.5.1
- new net B2: R17.1, ST1.3.1, U1.PWM6, X8.5.1
- new net B3: R21.1, ST2.3.1, U1.PWM10, X8.6.1
- new net B4: R25.1, ST3.3.1, U1.PWM14, X7.6.1
- new net D+: C8.1, IC2.USBDP, X1.D+
- new net D-: C7.1, IC2.USBDM, X1.D-
- new net G1: R11.1, U1.PWM1, X7.3.1
- new net G2: R15.1, ST1.2.1, U1.PWM5, X8.3.1
- new net G3: R19.1, ST2.2.1, U1.PWM9, X8.4.1
- new net G4: R23.1, ST3.2.1, U1.PWM13, X7.4.1
- new net N$15: Q7.D, X13.1, X9.5.1
- new net N$16: Q8.D, X9.6.1
- new net N$17: Q6.G, R15.2
- new net N$18: Q7.G, R16.2
- new net N$22: Q8.G, R17.2
- new net N$23: Q5.G, R14.2
- new net N$25: Q9.D, X14.1.1, X17.1
- new net N$26: Q10.D, X14.2.1
- new net N$27: Q11.D, X14.5.1, X18.1
- new net N$28: Q12.D, X14.6.1
- new net N$29: Q10.G, R19.2
- new net N$30: Q11.G, R20.2
- new net N$31: Q12.G, R21.2
- new net N$32: Q9.G, R18.2
- new net N$34: Q13.D, X19.1.1, X22.1
- new net N$35: Q14.D, X19.2.1
- new net N$36: Q15.D, X19.5.1, X23.1
- new net N$37: Q16.D, X19.6.1
- new net N$38: Q14.G, R23.2
- new net N$39: Q15.G, R24.2
- new net N$40: Q16.G, R25.2
- new net N$41: Q13.G, R22.2
- new net N$43: C2.1, D1.C, IC1.VIN
- new net R1: R10.2, U1.PWM0, X7.1.1
- new net R2: R14.1, ST1.1.1, U1.PWM4, X8.1.1
- new net R3: R18.1, ST2.1.1, U1.PWM8, X8.2.1
- new net R4: R22.1, ST3.1.1, U1.PWM12, X7.2.1
- new net W1: R12.1, U1.PWM3, X7.7.1
- new net W2: R16.1, ST1.4.1, U1.PWM7, X8.7.1
- new net W3: R20.1, ST2.4.1, U1.PWM11, X8.8.1
- new net W4: R24.1, ST3.4.1, U1.PWM15, X7.8.1
- net +12V: now also C11.+, C12.+, C13.+, D1.A, X10.1, X14.3.1, X14.4.1, X15.1, X19.3.1, X19.4.1, X2.3.1, X2.4.1, X20.1, X9.3.1, X9.4.1; no longer C5.1, IC1.VIN, X1.3.1, X1.4.1
- net +3V3: now also C10.1, C3.1, C4.+, R3.2, R4.2, R8.2, R9.2, U$1.VCC, U1.VDD; no longer C6.+, C7.1, C8.1, R19.2, R20.2, R21.2, R23.2, U$2.VCC, U2.VDD
- net +5V: now also C6.1, X1.VBUS; no longer C9.1, U$40.VBUS
- net GND: now also C10.2, C11.-, C12.-, C13.-, C4.-, C6.2, Q10.S, Q11.S, Q12.S, Q13.S, Q14.S, Q15.S, Q16.S, Q5.S, Q6.S, Q7.S, Q8.S, Q9.S, R5.1, ST1.5.1, ST2.5.1, ST3.5.1, U$1.GND, U1.#OE, U1.A0, U1.A1, U1.A2, U1.A3, U1.A4, U1.A5, U1.EXTCLK, U1.GND, X1.GND, X1.P$1, X1.P$2, X11.1, X16.1, X21.1, X7.10.1, X7.9.1, X8.10.1, X8.9.1; no longer C4.2, C6.-, R22.1, U$2.GND, U$40.GND, U$40.P$1, U$40.P$2, U2.#OE, U2.A0, U2.A1, U2.A2, U2.A3, U2.A4, U2.A5, U2.EXTCLK, U2.GND
- net GPIO0: now also R3.1, T1.C, U$1.GPIO0; no longer R23.1, T2.C, U$2.GPIO0
- net GPIO15: now also R5.2, U$1.GPIO15; no longer R22.2, U$2.GPIO15
- net N$1: now also X2.1.1; no longer X1.1.1
- net N$10: now also R7.2, T2.B; no longer R4.2, T1.B
- net N$11: now also R1.1, U$1.CH_PD; no longer R19.1, U$2.CH_PD
- net N$12: now also C9.1; no longer C2.1
- net N$13: now also R4.1, U$1.GPIO2; no longer R21.1, U$2.GPIO2
- net N$14: now also Q1.G, R10.1; no longer R5.2, U2.PWM0
- net N$19: now also Q2.G, R11.2; no longer R6.2, U2.PWM1
- net N$2: now also X2.2.1; no longer X1.2.1
- net N$20: now also Q3.G, R12.2; no longer R7.2, U2.PWM2
- net N$21: now also Q4.G, R13.2; no longer R8.2, U2.PWM3
- net N$3: now also Q5.D, X12.1, X9.1.1; no longer C4.1, IC2.USBDP, U$40.D+
- net N$4: now also X2.6.1; no longer X1.6.1
- net N$5: now also X2.5.1; no longer X1.5.1
- net N$6: now also Q6.D, X9.2.1; no longer C3.1, IC2.USBDM, U$40.D-
- net N$7: now also R6.1, T2.E; no longer R3.1, T1.E
- net N$8: now also R7.1, T1.E; no longer R4.1, T2.E
- net N$9: now also R6.2, T1.B; no longer R3.2, T2.B
- net RST: now also C5.1, R2.1, T2.C, U$1.GPIO18; no longer R20.1, T1.C, U$2.GPIO18
- net RX: now also U$1.URXD; no longer U$2.URXD
- net SCL: now also R9.1, U$1.GPIO12, U1.SCL; no longer R2.1, U$2.GPIO12, U2.SCL
- net SDA: now also R8.1, U$1.NC, U1.SDA; no longer R1.1, U$2.NC, U2.SDA
- net TX: now also U$1.UTXD; no longer U$2.UTXD
Other:
- note added: "Master Supply"
- note added: "RGBW Output 1"
- note added: "RGBW Output 2"
- note added: "RGBW Output 3"
- note added: "RGBW Output 4"
- note added: "Supply 2"
- note added: "Supply 3"
- note added: "Supply 4"
- note removed: "UART"
